File: kicad/p1p2_rs232_receiver.kicad_pcb (KiCad board)
At the start: 2 copper layers, 65 x 56.5 mm, 69 parts, among them J1 Raspberry_Pi_2_3, J2 PC MC_1,5_2-G-3.81, Q1 BSS123, SW1 SW_Push, U1 LM4040DBZ-3, U103 LM4871, U3 Pico

Commit message: kicad: Fixes for version v0.3
- Replace Ti LM4871 with STM TS4990
- Power SHUTDOWN from +5V rail
- Use double ground plane

Signed-off-by: Patrick Rudolph <rudolphpatrick05@gmail.com>
Parts:
- added Q2: BSS123, Package_TO_SOT_SMD:SOT-23, B.Cu at (69.1, 59.0)
- added R18: 10k, Resistor_SMD:R_0805_2012Metric_Pad1.20x1.40mm_HandSolder, B.Cu at (110.6, 48.0)
- added R19: 10k, Resistor_SMD:R_0805_2012Metric_Pad1.20x1.40mm_HandSolder, B.Cu at (106.6, 48.0)
- C8: footprint Capacitor_SMD:C_0603_1608Metric_Pad1.08x0.95mm_HandSolder -> Capacitor_SMD:C_0805_2012Metric_Pad1.18x1.45mm_HandSolder
- R104, R108: value 1k -> 4k7
- R14: value 47k -> 76k
- U103: value LM4871 -> TS4990
- moved R2 3.79 mm to (73.2, 59.4), turned to 180 degrees
- moved C113 1.79 mm to (66.6, 54.3)
- moved R11 1.18 mm to (77.1, 59.4)
- moved R12 0.80 mm to (80.5, 58.8)
- moved C3 0.21 mm to (116.3, 44.6)
Connections:
- R2 pad 1: +3V3 -> +VDC
- R2 pad 2: /SHUTDOWN -> Net-(R2-Pad2)
- U103 pad 1: /SHUTDOWN -> Net-(R2-Pad2)
Routing:
- net +3V3: track 1.91 -> 23.4 mm, vias 1 -> 3
- net Net-(R2-Pad2): track 0.00 -> 7.39 mm
- net Net-(D3-Pad1): track 95.8 -> 102.3 mm
- net Net-(C8-Pad1): track 4.83 -> 10.9 mm
- net Net-(C4-Pad2): track 111.9 -> 117.0 mm
- net +VDC: track 90.1 -> 93.5 mm
- net /SHUTDOWN: track 11.4 -> 10.6 mm
- net Net-(C113-Pad1): track 4.93 -> 5.67 mm
- net GND: vias 1 -> 12
- added copper zone on F.Cu, net GND
- removed copper zone on F.Cu, net +3V3
Other:
- board text added: "v0.3"
- board text removed: "v0.2"
